File: Amplifier-Concepts/Amplifier-Concepts.kicad_sch (KiCad schematic)
At the start: 0 parts

Commit message: updated concept
Parts:
- added Cant, Cant1, Cant2, Cant3, Cant4: 3p, symbol SLiCAP:C
- added N1, N2: ~, symbol SLiCAP:N
- added RLoad, RLoad1, Rin, Rin1, Rs, Rs1: 50, symbol SLiCAP:R
- added Rcomp: 60, symbol SLiCAP:R
- added Rcomp: 120, symbol SLiCAP:R
- added Rfb, Rfb1: 600, symbol SLiCAP:R
- added Rout: 300, symbol SLiCAP:R
- added TVS, TVS1: ~, symbol SLiCAP:D
- added Vant, Vant1: ?, symbol SLiCAP:V
Connections:
- new net: Cant.1, Rs.1, Vant.1 (p)
- new net: Cant4.2, N2.2 (outN), RLoad1.2, Rfb.1
- new net: Cant1.1, N1.3 (inp), Rin.2, Rout.2
- new net: Cant1.2, RLoad.1, Rcomp.2, Rout.1
- new net: Cant3.1, N2.3 (inp), Rfb1.2, Rin1.2
- new net: Cant3.2, RLoad1.1, Rcomp.2, Rfb1.1
- new net: Rin.1, Rs.2, TVS.2
- new net: N1.1 (outP), Rcomp.1
- new net: Cant2.1, Rs1.1, Vant1.1 (p)
- new net: N2.1 (outP), Rcomp.1
- new net: Rin1.1, Rs1.2, TVS1.2
- new net 0: Cant.2, Cant2.2, Cant4.1, N1.2 (outN), N1.4 (inN), N2.4 (inN), RLoad.2, Rfb.2, TVS.1, TVS1.1, Vant.2 (n), Vant1.2 (n)
