File: KiCad/Active_E_Field_Probe/TEST/TEST.kicad_sch (KiCad schematic)
At the start: 117 parts

Commit message: Latest Stuff
Parts:
- added C32, C34: {C_s}, symbol SLiCAP:C
- added C33, C35: {0.56*C_s}, symbol SLiCAP:C
- added R26, R27, R28, R29: 50, symbol SLiCAP:R
- added V12, V13: {V_in}, symbol SLiCAP:V
- added X24, X28, X31, X33: ~, symbol SLiCAP:M_noise
- added X25, X27, X29, X30, X34, X35: ~, symbol SLiCAP:XM
- added X26, X32: ~, symbol SLiCAP:XMD
Connections:
- net 0: now also R27.2, R29.2, V12.2 (n), V13.2 (n), X24.2 (comm), X25.1 (D), X25.2 (G), X25.4 (B), X27.2 (G), X27.4 (B), X28.1 (ext), X28.2 (comm), X29.3 (S), X29.4 (B), X30.3 (S), X30.4 (B), X31.2 (comm), X32.1 (D1), X33.1 (ext), X33.2 (comm), X34.3 (S), X34.4 (B), X35.3 (S), X35.4 (B)
- net Amp_out: now also C33.2, C35.2, R26.1, R28.1, X29.1 (D), X30.1 (D), X34.1 (D), X35.1 (D)
- net vo: now also R26.2, R27.1, R28.2, R29.1
- new net: X32.2 (D2), X34.2 (G), X35.2 (G)
- new net: X25.3 (S), X26.1 (D1)
- new net: X26.2 (D2), X27.3 (S)
- new net: X24.3 (int), X26.3 (G1)
- new net: X26.4 (G2), X28.3 (int)
- new net: X27.1 (D), X29.2 (G), X30.2 (G)
- new net: C32.2, C33.1, X24.1 (ext)
- new net: X32.4 (G2), X33.3 (int)
- new net: C34.2, C35.1, X31.1 (ext)
- new net: C32.1, V12.1 (p)
- new net: X31.3 (int), X32.3 (G1)
- new net: C34.1, V13.1 (p)
Other:
- moved on the sheet: C2, D1, F1, G1, N1, R2, V1

Commit message: STUFF
Parts:
- added C36: {C_s}, symbol SLiCAP:C
- added C37: {0.56*C_s}, symbol SLiCAP:C
- added R30: {R_ph}, symbol SLiCAP:R
- added R31, R32: 50, symbol SLiCAP:R
- added V14: {V_in}, symbol SLiCAP:V
- added X36, X40: ~, symbol SLiCAP:M_noise
- added X37, X39, X41, X42, X43, X44: ~, symbol SLiCAP:XM
- added X38: ~, symbol SLiCAP:XMD
Connections:
- net 0: now also R32.2, V14.2 (n), X36.2 (comm), X37.1 (D), X37.2 (G), X37.4 (B), X39.2 (G), X39.4 (B), X40.1 (ext), X40.2 (comm), X41.3 (S), X41.4 (B), X42.2 (G), X42.4 (B), X43.2 (G), X43.4 (B), X44.3 (S), X44.4 (B)
- net Amp_out: now also C37.2, X42.1 (D), X43.1 (D)
- net vo: now also R31.2, R32.1
- new net: C36.2, R30.1
- new net: C37.1, R30.2, X36.1 (ext)
- new net: X37.3 (S), X38.1 (D1)
- new net: X36.3 (int), X38.3 (G1)
- new net: C36.1, V14.1 (p)
- new net: R31.1, X43.3 (S), X44.1 (D)
- new net: X38.2 (D2), X39.3 (S)
- new net: X38.4 (G2), X40.3 (int)
- new net: X39.1 (D), X41.2 (G), X44.2 (G)
- new net: X41.1 (D), X42.3 (S)

Commit message: push
Parts:
- added C38: {C_s}, symbol SLiCAP:C
- added C39: {0.56*C_s}, symbol SLiCAP:C
- added R33: {R_ph}, symbol SLiCAP:R
- added R34, R35: 50, symbol SLiCAP:R
- added V15: {V_in}, symbol SLiCAP:V
- added X45, X49: ~, symbol SLiCAP:M_noise
- added X46, X48, X50, X51: ~, symbol SLiCAP:XM
- added X47: ~, symbol SLiCAP:XMD
Connections:
- net 0: now also R35.2, V15.2 (n), X45.2 (comm), X46.1 (D), X46.2 (G), X46.4 (B), X48.2 (G), X48.4 (B), X49.1 (ext), X49.2 (comm), X50.3 (S), X50.4 (B), X51.3 (S), X51.4 (B)
- net Amp_out: now also C39.2, R34.1, X50.1 (D), X51.1 (D)
- net vo: now also R34.2, R35.1
- new net: C39.1, R33.2, X45.1 (ext)
- new net: X45.3 (int), X47.3 (G1)
- new net: X48.1 (D), X50.2 (G), X51.2 (G)
- new net: X46.3 (S), X47.1 (D1)
- new net: X47.4 (G2), X49.3 (int)
- new net: X47.2 (D2), X48.3 (S)
- new net: C38.2, R33.1
- new net: C38.1, V15.1 (p)
