File: KiCad/Active_E_Field_Probe/Active_E_Field_Probe.kicad_sch (KiCad schematic)
At the start: 13 parts

Commit message: Fix shit
Parts:
- removed R1: 50, symbol SLiCAP:R
- X6, X7: W {220e-7} -> {W1_N}
Connections:
- net Amp_out: now also C23.2
Changed lines of the file:
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@@
 	(wire
 		(pts
-			(xy 171.45 39.37) (xy 186.69 39.37)
+			(xy 171.45 39.37) (xy 232.41 39.37)
 		)
 		(stroke
@@
 		(pts
 			(xy 210.82 49.53) (xy 210.82 68.58)
-		)
-		(stroke
-			(width 0)
-			(type default)
-		)
-	)
-	(wire
-		(pts
-			(xy 196.85 39.37) (xy 232.41 39.37)
 		)
 		(stroke
@@
 			)
 		)
-		(property "W" "{220e-7}"
+		(property "W" "{W1_N}"
 			(at 133.35 67.945 0)
 			(show_name yes)
@@
 				(path "/8648b04b-5135-4efe-a9b1-6520ac7dc88b"
 					(reference "X7")
-					(unit 1)
-				)
-			)
-		)
-	)
-	(symbol
-		(lib_id "SLiCAP:R")
-		(at 191.77 39.37 90)
-		(unit 1)
-		(exclude_from_sim no)
-		(in_bom yes)
-		(on_board yes)
-		(dnp no)
-		(property "Reference" "R1"
-			(at 192.278 30.734 90)
-			(effects
-				(font
-					(size 1.27 1.27)
-				)
-			)
-		)
-		(property "Value" "50"
-			(at 192.278 33.274 90)
-			(show_name yes)
-			(effects
-				(font
-					(size 1.27 1.27)
-				)
-			)
-		)
-		(property "Footprint" ""
-			(at 194.945 38.735 0)
-			(effects
-				(font
-					(size 1.27 1.27)
-				)
-				(hide yes)
-			)
-		)
-		(property "Datasheet" ""
-			(at 194.945 38.735 0)
-			(effects
-				(font
-					(size 1.27 1.27)
-				)
-				(hide yes)
-			)
-		)
-		(property "Description" "Resistor (cannot have zero resistance)"
-			(at 197.612 18.288 0)
-			(effects
-				(font
-					(size 1.27 1.27)
-				)
-				(hide yes)
-			)
-		)
-		(property "model" "R"
-			(at 195.58 37.465 0)
-			(show_name yes)
-			(effects
-				(font
-					(size 1.27 1.27)
-				)
-				(justify left)
-				(hide yes)
-			)
-		)
-		(property "noisetemp" "{T_op_max}"
-			(at 192.278 35.814 90)
-			(show_name yes)
-			(effects
-				(font
-					(size 1.27 1.27)
-				)
-			)
-		)
-		(property "noiseflow" "0"
-			(at 191.77 30.48 90)
-			(show_name yes)
-			(effects
-				(font
-					(size 1.27 1.27)
-				)
-				(hide yes)
-			)
-		)
-		(property "dcvar" "0"
-			(at 191.77 33.02 90)
-			(show_name yes)
-			(effects
-				(font
-					(size 1.27 1.27)
-				)
-				(hide yes)
-			)
-		)
-		(property "dcvarlot" "0"
-			(at 191.77 35.56 90)
-			(show_name yes)
-			(effects
-				(font
-					(size 1.27 1.27)
-				)
-				(hide yes)
-			)
-		)
-		(pin "2"
-		)
-		(pin "1"
-		)
-		(instances
-			(project "Active_E_Field_Probe"
-				(path "/8648b04b-5135-4efe-a9b1-6520ac7dc88b"
-					(reference "R1")
 					(unit 1)
 				)
@@
 		(dnp no)
 		(property "Reference" "X5"
-			(at 161.925 68.58 0)
+			(at 159.512 93.472 0)
 			(effects
 				(font
@@
 		)
 		(property "Value" "~"
-			(at 161.925 71.12 0)
+			(at 159.766 95.504 0)
 			(effects
 				(font
@@
 			)
 		)
-		(property "W" "{220e-7}"
+		(property "W" "{W1_N}"
 			(at 151.13 67.945 0)
 			(show_name yes)
@@
 		(on_board yes)
 		(dnp no)
-		(fields_autoplaced yes)
 		(property "Reference" "X4"
-			(at 122.555 68.58 0)
+			(at 126.238 93.218 0)
 			(effects
 				(font
@@
 		)
 		(property "Value" "~"
-			(at 122.555 71.12 0)
-			(effects
-				(font
+			(at 126.238 95.504 0)
+			(effects
+				(font

Commit message: Latest Stuff
Parts:
- removed C22: {C_s}, symbol SLiCAP:C
- removed C23: {0.56*C_s}, symbol SLiCAP:C
- removed R16, R17: 50, symbol SLiCAP:R
- removed X6, X7: ~, symbol SLiCAP:XM
- added C30: {C_s}, symbol SLiCAP:C
- added C31: {0.56*C_s}, symbol SLiCAP:C
- added R24, R25: 50, symbol SLiCAP:R
Connections:
- net 0: now also X1.1 (D1), R25.2
- net Amp_out: now also C31.2, R24.1
- net vo: now also R24.2, R25.1
- net at X4.1 (ext): now also C30.2, C31.1
- net at X2.2 (G), X3.2 (G): now also X1.2 (D2)
- net at V1.1 (p): now also C30.1

Commit message: More optimization stuff
Parts:
- added R1: {R_ph}, symbol SLiCAP:R
Connections:
- net at C31.1, X4.1 (ext): now also R1.2; no longer C30.2
- new net: C30.2, R1.1
Other:
- moved on the sheet: C30, V1
Changed lines of the file:
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@@
+	)
+	(junction
+		(at 81.28 86.36)
+		(diameter 0)
+		(color 0 0 0 0)
 	)
 	(junction
@@
 	)
 	(junction
-		(at 81.28 86.36)
-		(diameter 0)
-		(color 0 0 0 0)
-	)
-	(junction
 		(at 201.93 80.01)
 		(diameter 0)
@@
 	(wire
 		(pts
-			(xy 62.23 91.44) (xy 62.23 86.36)
+			(xy 50.8 93.98) (xy 50.8 86.36)
 		)
 		(stroke
@@
 	(wire
 		(pts
+			(xy 64.77 86.36) (xy 68.58 86.36)
+		)
+		(stroke
+			(width 0)
+			(type default)
+		)
+	)
+	(wire
+		(pts
 			(xy 180.34 100.33) (xy 180.34 106.68)
 		)
@@
 	(wire
 		(pts
-			(xy 62.23 86.36) (xy 68.58 86.36)
+			(xy 50.8 86.36) (xy 54.61 86.36)
 		)
 		(stroke
@@
 	(wire
 		(pts
+			(xy 78.74 86.36) (xy 81.28 86.36)
+		)
+		(stroke
+			(width 0)
+			(type default)
+		)
+	)
+	(wire
+		(pts
 			(xy 193.04 69.85) (xy 193.04 60.96)
 		)
@@
 	(wire
 		(pts
-			(xy 78.74 86.36) (xy 81.28 86.36)
-		)
-		(stroke
-			(width 0)
-			(type default)
-		)
-	)
-	(wire
-		(pts
 			(xy 180.34 106.68) (xy 184.15 106.68)
 		)
@@
 	(wire
 		(pts
-			(xy 62.23 101.6) (xy 62.23 106.68)
-		)
-		(stroke
-			(width 0)
-			(type default)
-		)
-	)
-	(wire
-		(pts
-			(xy 62.23 106.68) (xy 90.17 106.68)
+			(xy 50.8 104.14) (xy 50.8 106.68)
+		)
+		(stroke
+			(width 0)
+			(type default)
+		)
+	)
+	(wire
+		(pts
+			(xy 50.8 106.68) (xy 90.17 106.68)
 		)
 		(stroke
@@
 	)
 	(symbol
+		(lib_id "SLiCAP:R")
+		(at 73.66 86.36 90)
+		(unit 1)
+		(exclude_from_sim no)
+		(in_bom yes)
+		(on_board yes)
+		(dnp no)
+		(property "Reference" "R1"
+			(at 73.66 89.154 90)
+			(effects
+				(font
+					(size 1.27 1.27)
+				)
+			)
+		)
+		(property "Value" "{R_ph}"
+			(at 73.66 91.694 90)
+			(show_name yes)
+			(effects
+				(font
+					(size 1.27 1.27)
+				)
+			)
+		)
+		(property "Footprint" ""
+			(at 76.835 85.725 0)
+			(effects
+				(font
+					(size 1.27 1.27)
+				)
+				(hide yes)
+			)
+		)
+		(property "Datasheet" ""
+			(at 76.835 85.725 0)
+			(effects
+				(font
+					(size 1.27 1.27)
+				)
+				(hide yes)
+			)
+		)
+		(property "Description" "Resistor (cannot have zero resistance)"
+			(at 79.502 65.278 0)
+			(effects
+				(font
+					(size 1.27 1.27)
+				)
+				(hide yes)
+			)
+		)
+		(property "model" "R"
+			(at 77.47 84.455 0)
+			(show_name yes)
+			(effects
+				(font
+					(size 1.27 1.27)
+				)
+				(justify left)
+				(hide yes)
+			)
+		)
+		(property "noisetemp" "{T_op_max}"
+			(at 73.66 94.234 90)
+			(show_name yes)
+			(effects
+				(font
+					(size 1.27 1.27)
+				)
+			)
+		)
+		(property "noiseflow" "0"
+			(at 73.66 77.47 90)
+			(show_name yes)
+			(effects
+				(font
+					(size 1.27 1.27)
+				)
+				(hide yes)
+			)
+		)
+		(property "dcvar" "0"
+			(at 73.66 80.01 90)
+			(show_name yes)
+			(effects
+				(font
+					(size 1.27 1.27)
+				)
+				(hide yes)
+			)
+		)
+		(property "dcvarlot" "0"
+			(at 73.66 82.55 90)
+			(show_name yes)
+			(effects
+				(font
+					(size 1.27 1.27)
+				)
+				(hide yes)
+			)
+		)
+		(pin "1"
+		)
+		(pin "2"
+		)
+		(instances
+			(project ""
+				(path "/8648b04b-5135-4efe-a9b1-6520ac7dc88b"
+					(reference "R1")
+					(unit 1)
+				)
+			)
+		)
+	)
+	(symbol
 		(lib_id "SLiCAP:C")
-		(at 73.66 86.36 90)
+		(at 59.69 86.36 90)
 		(unit 1)
 		(exclude_from_sim no)
@@
 		(fields_autoplaced yes)
 		(property "Reference" "C30"
-			(at 73.5937 77.47 90)
+			(at 59.6237 77.47 90)
 			(effects
 				(font
@@
 		)
 		(property "Value" "{C_s}"
-			(at 73.5937 80.01 90)
+			(at 59.6237 80.01 90)
 			(show_name yes)
 			(effects
@@
 		)
 		(property "Footprint" ""
-			(at 74.93 83.82 0)
+			(at 60.96 83.82 0)
 			(effects
 				(font
@@
 		)
 		(property "Datasheet" ""
-			(at 74.93 83.82 0)
+			(at 60.96 83.82 0)
 			(effects
 				(font
@@
 		)
 		(property "Description" "Capacitor"
-			(at 79.756 79.248 0)
+			(at 65.786 79.248 0)
 			(effects
 				(font
@@
 		)
 		(property "model" "C"
-			(at 77.47 83.82 0)
+			(at 63.5 83.82 0)
 			(show_name yes)
 			(effects
@@
 		)
 		(property "vinit" "0"
-			(at 73.5937 82.55 90)
+			(at 59.6237 82.55 90)
 			(show_name yes)
 			(effects
@@
 	(symbol
 		(lib_id "SLiCAP:V")
-		(at 62.23 96.52 0)
+		(at 50.8 99.06 0)
 		(unit 1)
 		(exclude_from_sim no)
@@
 		(fields_autoplaced yes)
 		(property "Reference" "V1"
-			(at 66.04 95.1229 0)
+			(at 54.61 97.6629 0)
 			(effects
 				(font
@@
 		)
 		(property "Value" "{V_in}"
-			(at 66.04 97.6629 0)
+			(at 54.61 100.2029 0)
 			(show_name yes)
 			(effects
@@
 		)
 		(property "Footprint" ""
-			(at 62.23 97.79 0)
+			(at 50.8 100.33 0)
 			(effects
 				(font
@@
 		)
 		(property "Datasheet" ""
-			(at 62.23 97.79 0)
+			(at 50.8 100.33 0)
 			(effects
 				(font
@@
 		)
 		(property "Description" "Independent voltage source"
-			(at 78.74 103.632 0)
+			(at 67.31 106.172 0)
 			(effects
 				(font
@@
 		)
 		(property "noise" "0"
-			(at 66.04 98.9329 0)
+			(at 54.61 101.4729 0)
 			(show_name yes)
 			(effects
@@
 		)
 		(property "dc" "0"
-			(at 66.04 100.2029 0)
+			(at 54.61 102.7429 0)
 			(show_name yes)
 			(effects
@@
 		)
 		(property "dcvar" "0"
-			(at 66.04 101.4729 0)
+			(at 54.61 104.0129 0)
 			(show_name yes)
 			(effects
@@
 		)
 		(property "model" "V"
-			(at 65.405 101.6 0)
-			(show_name yes)
-			(effects
+			(at 53.975 104.14 0)
+			(show_name yes)
+			(effects

Commit message: cascode
Parts:
- added X6, X7: ~, symbol SLiCAP:XM
- renumbered C30 to C1, C31 to C2, R24 to R2, R25 to R3
Connections:
- net 0: now also X6.1 (D), X6.2 (G), X6.4 (B), X7.2 (G), X7.4 (B); no longer X1.1 (D1)
- net at X2.2 (G), X3.2 (G): now also X7.1 (D); no longer X1.2 (D2)
- new net: X1.2 (D2), X7.3 (S)
- new net: X1.1 (D1), X6.3 (S)
Other:
- moved on the sheet: C2, R2, R3, X2, X3

Commit message: STUFF
Parts:
- X6, X7: W {W1_N} -> {0.025*W1_N}
Changed lines of the file:
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@@
 			)
 		)
-		(property "W" "{W1_N}"
+		(property "W" "{0.025*W1_N}"
 			(at 120.65 65.405 0)
 			(show_name yes)
@@
 			)
 		)
-		(property "W" "{W1_N}"
+		(property "W" "{0.025*W1_N}"
 			(at 102.87 65.405 0)
 			(show_name yes)

Commit message: push
Parts:
- removed X5: ~, symbol SLiCAP:M_noise
- removed X6, X7: ~, symbol SLiCAP:XM
- added X4: ~, symbol SLiCAP:XM
- added X6: ~, symbol SLiCAP:M_noise
- renumbered X4 to X5
Connections:
- net 0: now also X1.1 (D1), X4.1 (D), X4.4 (B), X6.1 (ext), X6.2 (comm)
- net at X2.2 (G), X3.2 (G): now also X4.3 (S)
- net at X1.2 (D2): now also X4.2 (G)
- net at X1.4 (G2): now also X6.3 (int)
Other:
- moved on the sheet: C1, C2, R1, R2, R3, V1, X1, X2, X3, X5

Commit message: gemini
Parts:
- added X7, X8: ~, symbol SLiCAP:XM
Connections:
- net 0: now also X7.2 (G), X7.4 (B), X8.1 (D), X8.2 (G), X8.4 (B); no longer X1.1 (D1)
- net at X4.2 (G): now also X7.1 (D); no longer X1.2 (D2)
- new net: X1.1 (D1), X8.3 (S)
- new net: X1.2 (D2), X7.3 (S)

Commit message: 1st stage optim
Parts:
- removed R1: {R_ph}, symbol SLiCAP:R
- X7, X8: L {L1_N} -> {L1C_N}; W {0.1*W1_N} -> {W1C_N}
Connections:
- net at C2.1, X5.1 (ext): now also C1.2
Changed lines of the file:
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@@
+	)
+	(junction
+		(at 165.1 63.5)
+		(diameter 0)
+		(color 0 0 0 0)
 	)
 	(junction
@@
 	)
 	(junction
-		(at 181.61 46.99)
-		(diameter 0)
-		(color 0 0 0 0)
-	)
-	(junction
 		(at 105.41 106.68)
 		(diameter 0)
@@
 	(wire
 		(pts
-			(xy 165.1 46.99) (xy 165.1 66.04)
+			(xy 165.1 46.99) (xy 165.1 63.5)
 		)
 		(stroke
@@
 	(wire
 		(pts
-			(xy 181.61 46.99) (xy 198.12 46.99)
-		)
-		(stroke
-			(width 0)
-			(type default)
-		)
-	)
-	(wire
-		(pts
 			(xy 165.1 97.79) (xy 189.23 97.79)
 		)
@@
 	(wire
 		(pts
-			(xy 78.74 86.36) (xy 82.55 86.36)
+			(xy 78.74 86.36) (xy 95.25 86.36)
 		)
 		(stroke
@@
 	(wire
 		(pts
+			(xy 170.18 63.5) (xy 165.1 63.5)
+		)
+		(stroke
+			(width 0)
+			(type default)
+		)
+	)
+	(wire
+		(pts
 			(xy 119.38 46.99) (xy 119.38 58.42)
 		)
@@
 	(wire
 		(pts
-			(xy 165.1 46.99) (xy 181.61 46.99)
+			(xy 165.1 46.99) (xy 198.12 46.99)
 		)
 		(stroke
@@
 	(wire
 		(pts
-			(xy 92.71 86.36) (xy 95.25 86.36)
-		)
-		(stroke
-			(width 0)
-			(type default)
-		)
-	)
-	(wire
-		(pts
 			(xy 210.82 55.88) (xy 210.82 46.99)
 		)
@@
 	(wire
 		(pts
+			(xy 165.1 63.5) (xy 165.1 66.04)
+		)
+		(stroke
+			(width 0)
+			(type default)
+		)
+	)
+	(wire
+		(pts
+			(xy 170.18 71.12) (xy 170.18 63.5)
+		)
+		(stroke
+			(width 0)
+			(type default)
+		)
+	)
+	(wire
+		(pts
 			(xy 64.77 104.14) (xy 64.77 106.68)
 		)
@@
 	(wire
 		(pts
-			(xy 181.61 71.12) (xy 181.61 46.99)
-		)
-		(stroke
-			(width 0)
-			(type default)
-		)
-	)
-	(wire
-		(pts
 			(xy 64.77 106.68) (xy 105.41 106.68)
 		)
@@
 	(wire
 		(pts
-			(xy 165.1 71.12) (xy 181.61 71.12)
+			(xy 170.18 71.12) (xy 165.1 71.12)
 		)
 		(stroke
@@
 			)
 		)
-		(property "W" "{0.1*W1_N}"
+		(property "W" "{W1C_N}"
 			(at 118.11 65.405 0)
 			(show_name yes)
@@
 			)
 		)
-		(property "L" "{L1_N}"
+		(property "L" "{L1C_N}"
 			(at 118.11 67.945 0)
 			(show_name yes)
@@
 	)
 	(symbol
-		(lib_id "SLiCAP:R")
-		(at 87.63 86.36 90)
-		(unit 1)
-		(exclude_from_sim no)
-		(in_bom yes)
-		(on_board yes)
-		(dnp no)
-		(property "Reference" "R1"
-			(at 87.63 89.154 90)
-			(effects
-				(font
-					(size 1.27 1.27)
-				)
-			)
-		)
-		(property "Value" "{R_ph}"
-			(at 87.63 91.694 90)
-			(show_name yes)
-			(effects
-				(font
-					(size 1.27 1.27)
-				)
-			)
-		)
-		(property "Footprint" ""
-			(at 90.805 85.725 0)
-			(effects
-				(font
-					(size 1.27 1.27)
-				)
-				(hide yes)
-			)
-		)
-		(property "Datasheet" ""
-			(at 90.805 85.725 0)
-			(effects
-				(font
-					(size 1.27 1.27)
-				)
-				(hide yes)
-			)
-		)
-		(property "Description" "Resistor (cannot have zero resistance)"
-			(at 93.472 65.278 0)
-			(effects
-				(font
-					(size 1.27 1.27)
-				)
-				(hide yes)
-			)
-		)
-		(property "model" "R"
-			(at 91.44 84.455 0)
-			(show_name yes)
-			(effects
-				(font
-					(size 1.27 1.27)
-				)
-				(justify left)
-				(hide yes)
-			)
-		)
-		(property "noisetemp" "{T_op_max}"
-			(at 87.63 94.234 90)
-			(show_name yes)
-			(effects
-				(font
-					(size 1.27 1.27)
-				)
-			)
-		)
-		(property "noiseflow" "0"
-			(at 87.63 77.47 90)
-			(show_name yes)
-			(effects
-				(font
-					(size 1.27 1.27)
-				)
-				(hide yes)
-			)
-		)
-		(property "dcvar" "0"
-			(at 87.63 80.01 90)
-			(show_name yes)
-			(effects
-				(font
-					(size 1.27 1.27)
-				)
-				(hide yes)
-			)
-		)
-		(property "dcvarlot" "0"
-			(at 87.63 82.55 90)
-			(show_name yes)
-			(effects
-				(font
-					(size 1.27 1.27)
-				)
-				(hide yes)
-			)
-		)
-		(pin "1"
-		)
-		(pin "2"
-		)
-		(instances
-			(project ""
-				(path "/8648b04b-5135-4efe-a9b1-6520ac7dc88b"
-					(reference "R1")
-					(unit 1)
-				)
-			)
-		)
-	)
-	(symbol
 		(lib_id "SLiCAP:C")
 		(at 73.66 86.36 90)
@@
 			)
 		)
-		(property "W" "{0.1*W1_N}"
+		(property "W" "{W1C_N}"
 			(at 135.89 65.405 0)
 			(show_name yes)
@@
 			)
 		)
-		(property "L" "{L1_N}"
+		(property "L" "{L1C_N}"
 			(at 135.89 67.945 0)
 			(show_name yes)
