File: KiCad/Active_E_Field_Probe/stage_NP_PhZ_bias/Active_E_Field_Probe.kicad_sch (KiCad schematic)
At the start: 33 parts

Commit message: Biasing
Changed lines of the file:
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@@
 	(wire
 		(pts
-			(xy 214.63 41.91) (xy 214.63 46.99)
+			(xy 212.09 41.91) (xy 212.09 46.99)
 		)
 		(stroke
@@
 	(wire
 		(pts
+			(xy 212.09 41.91) (xy 214.63 41.91)
+		)
+		(stroke
+			(width 0)
+			(type default)
+		)
+	)
+	(wire
+		(pts
 			(xy 135.89 151.13) (xy 270.51 151.13)
 		)
@@
 		)
 		(stroke
-			(width 0)
-			(type default)
-		)
-	)
-	(wire
-		(pts
-			(xy 214.63 46.99) (xy 212.09 46.99)
-		)
-		(stroke
