File: KiCad/Active_E_Field_Probe/stage_N_balSF/Active_E_Field_Probe.kicad_sch (KiCad schematic)
At the start: 12 parts

Commit message: BW fix + bias initial
Changed lines of the file:
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@@
 	(paper "A4")
 	(junction
+		(at 190.5 67.31)
+		(diameter 0)
+		(color 0 0 0 0)
+	)
+	(junction
 		(at 121.92 93.98)
 		(diameter 0)
@@
 	)
 	(junction
-		(at 190.5 74.93)
-		(diameter 0)
-		(color 0 0 0 0)
-	)
-	(junction
 		(at 142.24 72.39)
 		(diameter 0)
@@
 	)
 	(junction
-		(at 195.58 106.68)
-		(diameter 0)
-		(color 0 0 0 0)
-	)
-	(junction
 		(at 210.82 86.36)
 		(diameter 0)
@@
 	)
 	(junction
+		(at 190.5 50.8)
+		(diameter 0)
+		(color 0 0 0 0)
+	)
+	(junction
 		(at 210.82 58.42)
 		(diameter 0)
@@
 	(wire
 		(pts
-			(xy 142.24 50.8) (xy 210.82 50.8)
+			(xy 142.24 50.8) (xy 190.5 50.8)
 		)
 		(stroke
@@
 	(wire
 		(pts
+			(xy 190.5 50.8) (xy 210.82 50.8)
+		)
+		(stroke
+			(width 0)
+			(type default)
+		)
+	)
+	(wire
+		(pts
 			(xy 210.82 86.36) (xy 217.17 86.36)
 		)
@@
 	(wire
 		(pts
+			(xy 210.82 63.5) (xy 210.82 58.42)
+		)
+		(stroke
+			(width 0)
+			(type default)
+		)
+	)
+	(wire
+		(pts
+			(xy 148.59 67.31) (xy 167.64 67.31)
+		)
+		(stroke
+			(width 0)
+			(type default)
+		)
+	)
+	(wire
+		(pts
+			(xy 142.24 50.8) (xy 142.24 72.39)
+		)
+		(stroke
+			(width 0)
+			(type default)
+		)
+	)
+	(wire
+		(pts
+			(xy 184.15 43.18) (xy 232.41 43.18)
+		)
+		(stroke
+			(width 0)
+			(type default)
+		)
+	)
+	(wire
+		(pts
+			(xy 232.41 74.93) (xy 210.82 74.93)
+		)
+		(stroke
+			(width 0)
+			(type default)
+		)
+	)
+	(wire
+		(pts
+			(xy 201.93 60.96) (xy 201.93 82.55)
+		)
+		(stroke
+			(width 0)
+			(type default)
+		)
+	)
+	(wire
+		(pts
+			(xy 190.5 90.17) (xy 190.5 82.55)
+		)
+		(stroke
+			(width 0)
+			(type default)
+		)
+	)
+	(wire
+		(pts
+			(xy 118.11 93.98) (xy 121.92 93.98)
+		)
+		(stroke
+			(width 0)
+			(type default)
+		)
+	)
+	(wire
+		(pts
+			(xy 236.22 74.93) (xy 232.41 74.93)
+		)
+		(stroke
+			(width 0)
+			(type default)
+		)
+	)
+	(wire
+		(pts
 			(xy 190.5 67.31) (xy 190.5 74.93)
 		)
@@
 	(wire
 		(pts
-			(xy 210.82 63.5) (xy 210.82 58.42)
-		)
-		(stroke
-			(width 0)
-			(type default)
-		)
-	)
-	(wire
-		(pts
-			(xy 148.59 67.31) (xy 167.64 67.31)
-		)
-		(stroke
-			(width 0)
-			(type default)
-		)
-	)
-	(wire
-		(pts
-			(xy 142.24 50.8) (xy 142.24 72.39)
-		)
-		(stroke
-			(width 0)
-			(type default)
-		)
-	)
-	(wire
-		(pts
-			(xy 184.15 43.18) (xy 232.41 43.18)
-		)
-		(stroke
-			(width 0)
-			(type default)
-		)
-	)
-	(wire
-		(pts
-			(xy 232.41 74.93) (xy 210.82 74.93)
-		)
-		(stroke
-			(width 0)
-			(type default)
-		)
-	)
-	(wire
-		(pts
-			(xy 195.58 106.68) (xy 210.82 106.68)
-		)
-		(stroke
-			(width 0)
-			(type default)
-		)
-	)
-	(wire
-		(pts
-			(xy 201.93 60.96) (xy 201.93 82.55)
-		)
-		(stroke
-			(width 0)
-			(type default)
-		)
-	)
-	(wire
-		(pts
-			(xy 190.5 90.17) (xy 190.5 82.55)
-		)
-		(stroke
-			(width 0)
-			(type default)
-		)
-	)
-	(wire
-		(pts
-			(xy 118.11 93.98) (xy 121.92 93.98)
-		)
-		(stroke
-			(width 0)
-			(type default)
-		)
-	)
-	(wire
-		(pts
-			(xy 236.22 74.93) (xy 232.41 74.93)
-		)
-		(stroke
-			(width 0)
-			(type default)
-		)
-	)
-	(wire
-		(pts
 			(xy 201.93 97.79) (xy 204.47 97.79)
 		)
@@
 	(wire
 		(pts
-			(xy 167.64 106.68) (xy 195.58 106.68)
+			(xy 167.64 106.68) (xy 210.82 106.68)
 		)
 		(stroke
@@
 	(wire
 		(pts
-			(xy 195.58 74.93) (xy 195.58 106.68)
-		)
-		(stroke
-			(width 0)
-			(type default)
-		)
-	)
-	(wire
-		(pts
 			(xy 104.14 104.14) (xy 104.14 106.68)
 		)
@@
 	(wire
 		(pts
+			(xy 190.5 50.8) (xy 190.5 67.31)
+		)
+		(stroke
+			(width 0)
+			(type default)
+		)
+	)
+	(wire
+		(pts
 			(xy 104.14 106.68) (xy 132.08 106.68)
 		)
@@
 		)
 		(stroke
-			(width 0)
-			(type default)
-		)
-	)
-	(wire
-		(pts
-			(xy 190.5 74.93) (xy 195.58 74.93)
-		)
-		(stroke

Commit message: Biasing
Parts:
- C2: value {0.56*C_s} -> {0.4*C_s}
Changed lines of the file:
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@@
 			)
 		)
-		(property "Value" "{0.56*C_s}"
+		(property "Value" "{0.4*C_s}"
 			(at 179.07 39.624 90)
 			(show_name yes)
