File: KiCad/Active_E_Field_Probe/stage_N_balSF_PhZ/Active_E_Field_Probe.kicad_sch (KiCad schematic)
At the start: 13 parts

Commit message: BW fix + bias initial
Changed lines of the file:
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@@
+	)
+	(junction
+		(at 190.5 59.69)
+		(diameter 0)
+		(color 0 0 0 0)
 	)
 	(junction
@@
 	)
 	(junction
-		(at 195.58 106.68)
-		(diameter 0)
-		(color 0 0 0 0)
-	)
-	(junction
 		(at 210.82 86.36)
 		(diameter 0)
@@
 	)
 	(junction
+		(at 190.5 46.99)
+		(diameter 0)
+		(color 0 0 0 0)
+	)
+	(junction
 		(at 210.82 100.33)
 		(diameter 0)
@@
 	)
 	(junction
-		(at 190.5 67.31)
-		(diameter 0)
-		(color 0 0 0 0)
-	)
-	(junction
 		(at 130.81 106.68)
 		(diameter 0)
@@
 	(wire
 		(pts
-			(xy 142.24 46.99) (xy 210.82 46.99)
+			(xy 142.24 46.99) (xy 190.5 46.99)
 		)
 		(stroke
@@
 	(wire
 		(pts
+			(xy 190.5 59.69) (xy 190.5 46.99)
+		)
+		(stroke
+			(width 0)
+			(type default)
+		)
+	)
+	(wire
+		(pts
 			(xy 204.47 53.34) (xy 201.93 53.34)
 		)
@@
 	(wire
 		(pts
-			(xy 195.58 106.68) (xy 210.82 106.68)
+			(xy 167.64 106.68) (xy 210.82 106.68)
 		)
 		(stroke
@@
 	(wire
 		(pts
-			(xy 167.64 106.68) (xy 195.58 106.68)
-		)
-		(stroke
-			(width 0)
-			(type default)
-		)
-	)
-	(wire
-		(pts
 			(xy 148.59 83.82) (xy 148.59 88.9)
 		)
@@
 	(wire
 		(pts
-			(xy 195.58 67.31) (xy 195.58 106.68)
-		)
-		(stroke
-			(width 0)
-			(type default)
-		)
-	)
-	(wire
-		(pts
 			(xy 85.09 104.14) (xy 85.09 106.68)
 		)
@@
 	(wire
 		(pts
-			(xy 190.5 67.31) (xy 195.58 67.31)
-		)
-		(stroke
+			(xy 190.5 46.99) (xy 210.82 46.99)
+		)
+		(stroke

Commit message: Biasing
Parts:
- C2: value {0.56*C_s} -> {0.4*C_s}
Changed lines of the file:
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@@
 			)
 		)
-		(property "Value" "{0.56*C_s}"
+		(property "Value" "{0.4*C_s}"
 			(at 161.29 43.434 90)
 			(show_name yes)
