File: KiCad/Active_E_Field_Probe/stage_PN/Active_E_Field_Probe.kicad_sch (KiCad schematic)
At the start: 14 parts

Commit message: diff vf
Parts:
- removed R1: {R_ph}, symbol SLiCAP:R
Connections:
- net at C2.1, X5.1 (ext): now also C1.2
Other:
- moved on the sheet: C1, C2, R2, R3, V1, X2, X3, X4

Commit message: BW fix + bias initial
Parts:
- X8: L {L1C_N} -> {L1C_P}; W {W1C_N} -> {W1C_P}
Changed lines of the file:
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@@
 			)
 		)
-		(property "W" "{W1C_N}"
+		(property "W" "{W1C_P}"
 			(at 119.38 80.645 0)
 			(show_name yes)
@@
 			)
 		)
-		(property "L" "{L1C_N}"
+		(property "L" "{L1C_P}"
 			(at 119.38 78.105 0)
 			(show_name yes)

Commit message: Biasing
Parts:
- C2: value {0.56*C_s} -> {0.4*C_s}
Changed lines of the file:
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@@
 			)
 		)
-		(property "Value" "{0.56*C_s}"
+		(property "Value" "{0.4*C_s}"
 			(at 160.782 28.702 90)
 			(show_name yes)
