File: KiCad/Active_E_Field_Probe/stage_P_balSF_PhZ/Active_E_Field_Probe.kicad_sch (KiCad schematic)
At the start: 13 parts

Commit message: Biasing
Parts:
- C2: value {0.56*C_s} -> {0.4*C_s}
Changed lines of the file:
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@@
 			)
 		)
-		(property "Value" "{0.56*C_s}"
+		(property "Value" "{0.4*C_s}"
 			(at 160.782 28.702 90)
 			(show_name yes)
